File: KiCad/tang-nano-9k-shield.kicad_sch (KiCad schematic)
At the start: 0 parts

Commit message: Add files via upload
Parts:
- added BZ1: Buzzer, symbol Device:Buzzer
- added C10, C11, C14, C22, C4, C5, C9: 100nF, symbol Device:C_Small
- added C12, C13: 2.2nF, symbol Device:C_Small
- added C15, C2, C3, C8: 10uF, symbol Device:C_Small
- added C16, C17: 1uF, symbol Device:C_Small
- added C18, C19: 47pF, symbol Device:C_Small
- added C20, C21: 100uF, symbol Device:C_Small
- added C6, C7: 22uF, symbol Device:C_Small
- added D1: SS14, Diode_SMD:D_SMA, symbol Diode:SS14
- added D2: 1N4148W, Diode_SMD:D_SOD-123, symbol Diode:1N4148W
- added J1: Barrel_Jack, symbol Connector:Barrel_Jack
- added J2: AudioJack3, symbol Connector_Audio:AudioJack3
- added L1: 3.3uH, symbol Device:L_Small
- added Q1: SS8050, Package_TO_SOT_SMD:SOT-23, symbol Transistor_BJT:SS8050
- added R1, R2, R3, R4: 4K7, symbol Device:R_Small
- added R10, R11, R5, R9: 330R, symbol Device:R_Small
- added R12, R13: 47R, symbol Device:R_Small
- added R14, R15, R16, R17, R21, R6, R8: 10K, symbol Device:R_Small
- added R18: 1K, symbol Device:R_Small
- added R19, R20: 20K, symbol Device:R_Small
- added R7: 54K9, symbol Device:R_Small
- added U1: Tang Nano 9K, symbol TangNano9K:Tang-Nano-9K
- added U2: (no value), symbol TangNano9K:Dual-PS/2
- added U3: TPS563201DDCR, TPS563201DDCR:SOT95P280X110-6N, symbol TPS563201DDCR:TPS563201DDCR
- added U4: AMS1117-3.3, Package_TO_SOT_SMD:SOT-223-3_TabPin2, symbol Regulator_Linear:AMS1117-3.3
- added U5: PT8211, PT8211:SOP8-6.0-4.9X3.9, symbol PT8211:PT8211
- added U6: LMV358, symbol Amplifier_Operational:LMV358
Connections:
- new net: R5.1, U2.1
- new net: C15.1, R14.2, R15.1, U6.3 (+), U6.5 (+)
- new net: C18.1, R17.2, R19.1, U6.6 (-)
- new net: C18.2, C21.1, R19.2, U6.7
- new net: C2.1, C3.1, C4.1, D1.1 (K), R6.2, U3.3 (VIN)
- new net: R13.1, U5.6 (LCH)
- new net: R6.1, U3.5 (EN)
- new net: R10.1, U2.7
- new net: C16.2, R16.1
- new net: C19.1, R16.2, R20.1, U6.2 (-)
- new net: R9.1, U2.11
- new net: R11.1, U2.5
- new net: Q1.1 (B), R18.2
- new net: C5.1, L1.1, U3.2 (SW)
- new net: D1.2 (A), J1.1
- new net: C5.2, U3.6 (VBST)
- new net: C17.2, R17.1
- new net: C19.2, C20.1, R20.2, U6.1
- new net: C21.2, J2.R
- new net: BZ1.2 (-), D2.2 (A), Q1.3 (C)
- new net: R12.1, U5.8 (RCH)
- new net: R7.2, R8.1, U3.4 (VFB)
- new net: C20.2, J2.T
- new net 3V3: C8.1, C9.1, R1.1, R2.1, R3.1, R4.1, U4.2 (VO)
- new net 5V: BZ1.1 (+), C10.1, C11.1, C14.1, C22.1, C6.1, C7.1, D2.1 (K), L1.2, R14.1, R7.1, U1.5V, U2.10, U2.4, U4.3 (VI), U5.5 (VDD), U6.8 (V+)
- new net BCK: U1.51 (IOR17B), U5.1 (BCK)
- new net BUZ: R18.1, R21.2, U1.38 (IOB31B)
- new net DIN: U1.54 (IOR15A), U5.3 (DIN)
- new net GND: C10.2, C11.2, C12.2, C13.2, C14.2, C15.2, C2.2, C22.2, C3.2, C4.2, C6.2, C7.2, C8.2, C9.2, J1.2, J2.S, Q1.2 (E), R15.2, R21.1, R8.2, U1.GND, U2.3, U2.9, U2.MP, U3.1 (GND), U4.1 (GND), U5.4 (GND), U6.4 (V-)
- new net LCH: C13.1, C16.1, R13.2
- new net PS/2_CLK1: R1.2, R11.2, U1.71 (IOT41A)
- new net PS/2_CLK2: R3.2, R9.2, U1.48 (IOR24B)
- new net PS/2_DAT1: R2.2, R5.2, U1.70 (IOT41B)
- new net PS/2_DAT2: R10.2, R4.2, U1.49 (IOR24A)
- new net RCH: C12.1, C17.1, R12.2
- new net WS: U1.53 (IOR15B), U5.2 (WS)
- no-connect marks 0 -> 5
Other:
- note added: "AUDIO"
- note added: "Left"
- note added: "POWER"
- note added: "PS/2"
- note added: "Right"

Commit message: Add files via upload
Parts:
- removed C21: 100uF, symbol Device:C_Small
- removed R14, R15, R16, R17: 10K, symbol Device:R_Small
- removed R19, R20: 20K, symbol Device:R_Small
- removed U6: LMV358, symbol Amplifier_Operational:LMV358
- added U6: TPA6132A2RTE, Package_DFN_QFN:WQFN-16-1EP_3x3mm_P0.5mm_EP1.6x1.6mm_ThermalVias, symbol Amplifier_Audio:TPA6132A2RTE
- C14: value 100nF -> 1uF
- C15: value 10uF -> 2.2uF
- C18, C19: value 47pF -> 1uF
- C20: value 100uF -> 1uF
Connections:
- net 5V: now also C14.2, U6.13 (EN), U6.14 (VDD), U6.6 (G0); no longer C14.1
- net GND: now also C14.1, C15.1, C18.1, C20.1, U6.10 (PGND), U6.15 (SGND), U6.17 (EP), U6.7 (G1); no longer C14.2, C15.2
- net at C18.2: now also U6.2 (INL+), U6.3 (INR+)
- net at C16.2: now also U6.1 (INL-)
- net at C19.1: now also U6.9 (CPN)
- net at C17.2: now also U6.4 (INR-)
- net at C19.2: now also U6.11 (CPP); no longer C20.1
- net at J2.R: now also U6.5 (OUTR)
- net at J2.T: now also U6.16 (OUTL); no longer C20.2
- new net: C20.2, U6.8 (HPVSS)
- new net: C15.2, U6.12 (HPVDD)
Other:
- note removed: "Left"
- note removed: "Right"
- moved on the sheet: BZ1, C11, C12, C13, D2, J2, Q1, R12, R13, R18, R21

Commit message: Add files via upload
Parts:
- added C23, C24: 100nF, symbol Device:C_Small
- added J3: USB_A_Stacked, symbol Connector:USB_A_Stacked
- added J5: DE15_Socket_HighDensity_MountingHoles, symbol Connector:DE15_Socket_HighDensity_MountingHoles
- added R14, R15: 100R, symbol Device:R_Small
- added R16, R22, R26: 510R, symbol Device:R_Small
- added R17, R23, R27: 1K, symbol Device:R_Small
- added R19, R24, R28: 2K, symbol Device:R_Small
- added R20, R25, R29: 3K9, symbol Device:R_Small
- added U7, U8: USBLC6-2SC6, Package_TO_SOT_SMD:SOT-23-6, symbol Power_Protection:USBLC6-2SC6
Connections:
- net 5V: now also C23.1, C24.1, J3.1 (VBUS1), J3.5 (VBUS2), U7.5 (VBUS), U8.5 (VBUS)
- net GND: now also C23.2, C24.2, J3.4 (GND1), J3.8 (GND2), J3.SH (Shield), J5.10, J5.5, J5.6, J5.7, J5.8, J5.SH, U7.2 (GND), U8.2 (GND)
- net VGA_VS: now reaches U1.72 (IOT39B)
- net VGA_VS: now also R15.2
- net VGA_HS: now reaches U1.73 (IOT39A)
- net VGA_HS: now also R14.2
- net VGA_B3: now reaches U1.74 (IOT38B)
- net VGA_B3: now also R26.1
- net VGA_B2: now reaches U1.75 (IOT38A)
- net VGA_B2: now also R27.1
- net VGA_B1: now reaches U1.76 (IOT37B)
- net VGA_B1: now also R28.1
- net VGA_B0: now reaches U1.77 (IOT37A)
- net VGA_B0: now also R29.1
- net VGA_G3: now reaches U1.79 (IOT12B)
- net VGA_G3: now also R22.1
- net VGA_G2: now reaches U1.80 (IOT12A)
- net VGA_G2: now also R23.1
- net VGA_G1: now reaches U1.81 (IOT11B)
- net VGA_G1: now also R24.1
- net VGA_G0: now reaches U1.82 (IOT11A)
- net VGA_G0: now also R25.1
- net VGA_R3: now reaches U1.83 (IOT10B)
- net VGA_R3: now also R16.1
- net VGA_R2: now reaches U1.84 (IOT10A)
- net VGA_R2: now also R17.1
- net VGA_R1: now reaches U1.85 (IOT8B)
- net VGA_R1: now also R19.1
- net VGA_R0: now reaches U1.86 (IOT8A)
- net VGA_R0: now also R20.1
- new net: J5.13, R14.1
- new net: J5.14, R15.1
- new net BLUE: J5.3, R26.2, R27.2, R28.2, R29.2
- new net D1+: U7.6 (I/O1)
- new net D1-: U7.4 (I/O2)
- new net D2+: U8.6 (I/O1)
- new net D2-: U8.4 (I/O2)
- new net GREEN: J5.2, R22.2, R23.2, R24.2, R25.2
- new net RAW_D1+: J3.3 (D1+), U7.1 (I/O1)
- new net RAW_D1-: J3.2 (D1-), U7.3 (I/O2)
- new net RAW_D2+: J3.7 (D2+), U8.1 (I/O1)
- new net RAW_D2-: J3.6 (D2-), U8.3 (I/O2)
- new net RED: J5.1, R16.2, R17.2, R19.2, R20.2
- no-connect marks 5 -> 10
Other:
- note added: "VGA"
- moved on the sheet: BZ1, C11, C12, C13, C14, C15, C16, C17, C18, C19, C20, D2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

Commit message: Add files via upload
Parts:
- removed J3: USB_A_Stacked, symbol Connector:USB_A_Stacked
- removed U8: USBLC6-2SC6, Package_TO_SOT_SMD:SOT-23-6, symbol Power_Protection:USBLC6-2SC6
- added C1, C21: 20pF, symbol Device:C_Small
- added C25, C26, C27, C28, C29, C30: 100nF, symbol Device:C_Small
- added D3, D4: SS14, Diode_SMD:D_SMA, symbol Diode:SS14
- added J3: USB_C_Receptacle_USB2.0_16P, symbol Connector:USB_C_Receptacle_USB2.0_16P
- added J6: DE9_Socket_MountingHoles, symbol Connector:DE9_Socket_MountingHoles
- added JP1: SolderJumper_2_Open, symbol Jumper:SolderJumper_2_Open
- added JP2: RST, symbol Jumper:SolderJumper_2_Open
- added R30: 10K, symbol Device:R_Small
- added R31, R32: 5K1, symbol Device:R_Small
- added U10: MAX3232, symbol Interface_UART:MAX3232
- added U8: RP2040, Package_DFN_QFN:QFN-56-1EP_7x7mm_P0.4mm_EP3.2x3.2mm, symbol MCU_RaspberryPi:RP2040
- added U9: W25Q32JVZP, Package_SON:WSON-8-1EP_6x5mm_P1.27mm_EP3.4x4.3mm, symbol Memory_Flash:W25Q32JVZP
- added Y1: X322512MSB4SI, symbol Device:Crystal_GND23_Small
Connections:
- net 3V3: now also C23.2, C25.2, R30.1, U10.16 (VCC), U8.1 (IOVDD), U8.10 (IOVDD), U8.22 (IOVDD), U8.33 (IOVDD), U8.42 (IOVDD), U8.43 (ADC_AVDD), U8.44 (VREG_VIN), U8.48 (USB_VDD), U8.49 (IOVDD), U9.8 (VCC)
- net 5V: now also D3.1 (K), D4.1 (K); no longer C23.1, C6.1, C7.1, L1.2, R7.1
- net D1+: now also U8.47 (USB_DP)
- net D1-: now also U8.46 (USB_DM)
- net GND: now also C23.1, C1.1, C21.1, C25.1, C26.1, C29.2, C30.2, J3.A1 (GND), J3.A12 (GND), J3.B1 (GND), J3.B12 (GND), J3.SH (SHIELD), J6.5, J6.SH (PAD), JP1.1 (A), JP2.1 (A), R31.2, R32.2, U10.15 (GND), U8.57 (GND), U9.4 (GND), U9.9 (EP), Y1.2 (G), Y1.3 (G); no longer C23.2
- net RAW_D1+: now also J3.A6 (D+), J3.B6 (D+)
- net RAW_D1-: now also J3.A7 (D-), J3.B7 (D-)
- net SCK: now reaches U1.28 (IOB11B)
- net SCK: now also U8.29 (GPIO18)
- net MOSI: now reaches U1.29 (IOB13A)
- net MOSI: now also U8.27 (GPIO16)
- net MISO: now reaches U1.30 (IOB13B)
- net MISO: now also U8.30 (GPIO19)
- net CS1: now reaches U1.33 (IOB23A)
- net CS1: now also U8.28 (GPIO17)
- net INT1: now reaches U1.34 (IOB23B)
- net INT1: now also U8.31 (GPIO20)
- net RS_RX: now reaches U1.36 (IOB29B)
- net RS_RX: now also U10.12 (R1OUT)
- net RS_TX: now reaches U1.37 (IOB31A)
- net RS_TX: now also U10.11 (T1IN)
- new net: C28.1, U10.4 (C2+)
- new net: C28.2, U10.5 (C2-)
- new net: C26.2, U8.23 (DVDD), U8.45 (VREG_VOUT), U8.50 (DVDD)
- new net: JP2.2 (B), R30.2, U8.26 (RUN)
- new net: U8.51 (QSPI_SD3), U9.7 (~{HOLD}/~{RESET}/IO_{3})
- new net: U8.52 (QSPI_SCLK), U9.6 (CLK)
- new net: U8.53 (QSPI_SD0), U9.5 (DI/IO_{0})
- new net: U8.54 (QSPI_SD2), U9.3 (~{WP}/IO_{2})
- new net: U8.55 (QSPI_SD1), U9.2 (DO/IO_{1})
- new net: J3.A5 (CC1), R31.1
- new net: C29.1, U10.2 (VS+)
- new net: C30.1, U10.6 (VS-)
- new net: J3.B5 (CC2), R32.1
- new net: C27.1, U10.1 (C1+)
- new net: C27.2, U10.3 (C1-)
- new net 5V_BUCK: C6.1, C7.1, D4.2 (A), L1.2, R7.1
- new net 5V_USB: D3.2 (A), J3.A4 (VBUS), J3.A9 (VBUS), J3.B4 (VBUS), J3.B9 (VBUS)
- new net BOOTSEL: JP1.2 (B), U8.56 (~{QSPI_SS}), U9.1 (~{CS})
- new net RXD: J6.2, U10.14 (T1OUT)
- new net TXD: J6.3, U10.13 (R1IN)
- new net XIN: C1.2, U8.20 (XIN), Y1.1
- new net XOUT: C21.2, U8.21 (XOUT), Y1.4
- no-connect marks 10 -> 50
Other:
- note added: "RP 2040"
- note added: "RS-232"
- note added: "USB-C"
- moved on the sheet: BZ1, C10, C11, C12, C13, C14, C15, C16, C17, C18, C19, C2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

Commit message: Add files via upload
Parts:
- added J4: I2C_headers, symbol Connector:Conn_01x04_Socket
- added J7: SPI_headers, symbol Connector:Conn_01x07_Socket
- added R33, R34, R35, R36: 10K, symbol Device:R_Small
- added SW1: RotaryEncoder_Switch_MP, symbol Device:RotaryEncoder_Switch_MP
- added SW2, SW3, SW4: SW_Push, symbol Switch:SW_Push
Connections:
- net 3V3: now also J4.2 (Pin_2), J7.2 (Pin_2), R33.1, R34.1, R35.1, R36.1
- net BCK: no longer U1.51 (IOR17B)
- net BUZ: no longer U1.38 (IOB31B)
- net CS1: no longer U1.33 (IOB23A)
- net DIN: no longer U1.54 (IOR15A)
- net GND: now also J4.1 (Pin_1), J7.1 (Pin_1), SW1.C, SW1.MP, SW1.S2, SW2.1, SW3.1, SW4.1
- net INT1: no longer U1.34 (IOB23B)
- net MISO: now also J7.5 (Pin_5); no longer U1.30 (IOB13B)
- net MOSI: now also J7.4 (Pin_4); no longer U1.29 (IOB13A)
- net PS/2_CLK1: no longer U1.71 (IOT41A)
- net PS/2_CLK2: no longer U1.48 (IOR24B)
- net PS/2_DAT1: no longer U1.70 (IOT41B)
- net PS/2_DAT2: no longer U1.49 (IOR24A)
- net RS_RX: no longer U1.36 (IOB29B)
- net RS_TX: no longer U1.37 (IOB31A)
- net SCK: now also J7.3 (Pin_3); no longer U1.28 (IOB11B)
- net VGA_B0: no longer U1.77 (IOT37A)
- net VGA_B1: no longer U1.76 (IOT37B)
- net VGA_B2: no longer U1.75 (IOT38A)
- net VGA_B3: no longer U1.74 (IOT38B)
- net VGA_G0: no longer U1.82 (IOT11A)
- net VGA_G1: no longer U1.81 (IOT11B)
- net VGA_G2: no longer U1.80 (IOT12A)
- net VGA_G3: no longer U1.79 (IOT12B)
- net VGA_HS: no longer U1.73 (IOT39A)
- net VGA_R0: no longer U1.86 (IOT8A)
- net VGA_R1: no longer U1.85 (IOT8B)
- net VGA_R2: no longer U1.84 (IOT10A)
- net VGA_R3: no longer U1.83 (IOT10B)
- net VGA_VS: no longer U1.72 (IOT39B)
- net WS: no longer U1.53 (IOR15B)
- new net CS2: J7.6 (Pin_6)
- new net ENC_A: SW1.A
- new net ENC_B: SW1.B
- new net ENC_SW: R33.2, SW1.S1
- new net INT2: J7.7 (Pin_7)
- new net SCL: J4.4 (Pin_4)
- new net SDA: J4.3 (Pin_3)
- new net SW1: R36.2, SW2.2
- new net SW2: R35.2, SW3.2
- new net SW3: R34.2, SW4.2
- no-connect marks 50 -> 68
Other:
- moved on the sheet: C22, U1

Commit message: Add files via upload
Parts:
- removed R33: 10K, symbol Device:R_Small
- removed SW1: RotaryEncoder_Switch_MP, symbol Device:RotaryEncoder_Switch_MP
- removed SW2, SW3, SW4: SW_Push, symbol Switch:SW_Push
- added C31, C33: 100nF, symbol Device:C_Small
- added C32: 10uF, symbol Device:C_Small
- added R37, R38: 4K7, symbol Device:R_Small
- added R39, R40, R41, R42, R43: 10K, symbol Device:R_Small
- added SW2: SW_DIP_x08, symbol Switch:SW_DIP_x08
- added U11: AMS1117-1.8, Package_TO_SOT_SMD:SOT-223-3_TabPin2, symbol Regulator_Linear:AMS1117-1.8
Connections:
- net 3V3: now also C31.1, R37.1, R38.1, U11.3 (VI); no longer R34.1, R35.1, R36.1
- net BCK: now also U1.74 (IOT38B)
- net BUZ: now also U1.75 (IOT38A)
- net CS1: now also U1.25 (IOB8A)
- net CS2: now also U1.27 (IOB11A)
- net DIN: now also U1.72 (IOT39B)
- net GND: now also C31.2, C32.2, C33.2, SW2.10, SW2.11, SW2.12, SW2.13, SW2.14, SW2.15, SW2.16, SW2.9, U11.1 (GND)
- net INT1: now also U1.26 (IOB8B)
- net INT2: now also U1.28 (IOB11B)
- net MISO: now also U1.39 (IOB33A)
- net MOSI: now also U1.37 (IOB31A)
- net PS/2_CLK1: now also U1.48 (IOR24B)
- net PS/2_CLK2: now also U1.31 (IOB15A)
- net PS/2_DAT1: now also U1.49 (IOR24A)
- net PS/2_DAT2: now also U1.32 (IOB15B)
- net RS_RX: now also U1.70 (IOT41B)
- net RS_TX: now also U1.71 (IOT41A)
- net SCK: now also U1.36 (IOB29B)
- net SCL: now also U1.69 (IOT42A), R37.2
- net SDA: now also U1.68 (IOT42B), R38.2
- net SW1: now also R34.2, U1.86 (IOT8A), SW2.1; no longer R36.2
- net SW2: now also U1.85 (IOT8B), SW2.2
- net SW3: now also R36.2, U1.84 (IOT10A), SW2.3; no longer R34.2
- net VGA_B0: now also U1.35 (IOB29A)
- net VGA_B1: now also U1.40 (IOB33B)
- net VGA_B2: now also U1.34 (IOB23B)
- net VGA_B3: now also U1.33 (IOB23A)
- net VGA_G0: now also U1.56 (IOR14A)
- net VGA_G1: now also U1.57 (IOR13A)
- net VGA_G2: now also U1.55 (IOR14B)
- net VGA_G3: now also U1.54 (IOR15A)
- net VGA_HS: now also U1.30 (IOB13B)
- net VGA_R0: now also U1.53 (IOR15B)
- net VGA_R1: now also U1.51 (IOR17B)
- net VGA_R2: now also U1.42 (IOB41B)
- net VGA_R3: now also U1.41 (IOB41A)
- net VGA_VS: now also U1.29 (IOB13A)
- net WS: now also U1.73 (IOT39A)
- net SW8: now reaches U1.79 (IOT12B)
- net SW8: now also R43.2, SW2.8
- net SW7: now reaches U1.80 (IOT12A)
- net SW7: now also R42.2, SW2.7
- net SW6: now reaches U1.81 (IOT11B)
- net SW6: now also R41.2, SW2.6
- net SW5: now reaches U1.82 (IOT11A)
- net SW5: now also R40.2, SW2.5
- net SW4: now reaches U1.83 (IOT10B)
- net SW4: now also R39.2, SW2.4
- new net 1V8: C32.1, C33.1, R34.1, R35.1, R36.1, R39.1, R40.1, R41.1, R42.1, R43.1, U11.2 (VO)
- no-connect marks 68 -> 54
Other:
- note added: "DIP Switches"
- note added: "Extension headers"
- note added: "Tang Nano"
- moved on the sheet: C10, C2, C22, C3, C4, C5, C6, C7, C8, C9, D1, D3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

Commit message: Add files via upload
Parts:
- BZ1: footprint (none) -> Buzzer_Beeper:MagneticBuzzer_ProSignal_ABT-410-RC
- C1: renamed from C10; footprint (none) -> Capacitor_SMD:C_0603_1608Metric
- C10: renamed from C12; footprint (none) -> Capacitor_SMD:C_0603_1608Metric
- C11: renamed from C13; footprint (none) -> Capacitor_SMD:C_0603_1608Metric
- C12: renamed from C17; footprint (none) -> Capacitor_SMD:C_0603_1608Metric
- C13: renamed from C16; footprint (none) -> Capacitor_SMD:C_0603_1608Metric
- C14: renamed from C5; footprint (none) -> Capacitor_SMD:C_0603_1608Metric
- C15: renamed from C14; footprint (none) -> Capacitor_SMD:C_0603_1608Metric
- C16: renamed from C20; footprint (none) -> Capacitor_SMD:C_0603_1608Metric
- C17: renamed from C7; footprint (none) -> Capacitor_SMD:C_1206_3216Metric
- C18: renamed from C15; footprint (none) -> Capacitor_SMD:C_0603_1608Metric
- C19: renamed from C6; footprint (none) -> Capacitor_SMD:C_1206_3216Metric
- C2, C3: footprint (none) -> Capacitor_SMD:C_1206_3216Metric
- C20: renamed from C19; footprint (none) -> Capacitor_SMD:C_0603_1608Metric
- C21: renamed from C31; footprint (none) -> Capacitor_SMD:C_0603_1608Metric
- C22: renamed from C32; footprint (none) -> Capacitor_SMD:C_1206_3216Metric
- C23: renamed from C33; footprint (none) -> Capacitor_SMD:C_0603_1608Metric
- C24: renamed from C27; footprint (none) -> Capacitor_SMD:C_0603_1608Metric
- C25, C4: footprint (none) -> Capacitor_SMD:C_0603_1608Metric
- C26: renamed from C1; footprint (none) -> Capacitor_SMD:C_0603_1608Metric
- C27: renamed from C24; footprint (none) -> Capacitor_SMD:C_0603_1608Metric
- C28: renamed from C23; footprint (none) -> Capacitor_SMD:C_0603_1608Metric
- C29: renamed from C21; footprint (none) -> Capacitor_SMD:C_0603_1608Metric
- C30: renamed from C28; footprint (none) -> Capacitor_SMD:C_0603_1608Metric
- C31: renamed from C29; footprint (none) -> Capacitor_SMD:C_0603_1608Metric
- C32: renamed from C30; footprint (none) -> Capacitor_SMD:C_0603_1608Metric
- C33: renamed from C26; footprint (none) -> Capacitor_SMD:C_0603_1608Metric
- C5: renamed from C22; footprint (none) -> Capacitor_SMD:C_0603_1608Metric
- C6: renamed from C8; footprint (none) -> Capacitor_SMD:C_1206_3216Metric
- C7: renamed from C9; footprint (none) -> Capacitor_SMD:C_0603_1608Metric
- C8: renamed from C11; footprint (none) -> Capacitor_SMD:C_0603_1608Metric
- C9: renamed from C18; footprint (none) -> Capacitor_SMD:C_0603_1608Metric
- J1: footprint (none) -> Connector_BarrelJack:BarrelJack_CLIFF_FC681465S_SMT_Horizontal
- J2: renamed from J5; footprint (none) -> Connector_Dsub:DSUB-15-HD_Pins_Horizontal_P2.29x2.54mm_EdgePinOffset8.35mm_Housed_MountingHolesOffset10.89mm
- J3: renamed from J4; footprint (none) -> Connector_PinHeader_2.54mm:PinHeader_1x04_P2.54mm_Vertical
- J4: renamed from J2; footprint (none) -> Connector_Audio:Jack_3.5mm_KoreanHropartsElec_PJ-320D-4A_Horizontal
- J5: renamed from J7; footprint (none) -> Connector_PinHeader_2.54mm:PinHeader_1x07_P2.54mm_Vertical
- J6: renamed from J3; footprint (none) -> Connector_USB:USB_C_Receptacle_G-Switch_GT-USB-7010ASV
- J7: renamed from J6; footprint (none) -> Connector_Dsub:DSUB-9_Pins_Horizontal_P2.77x2.84mm_EdgePinOffset7.70mm_Housed_MountingHolesOffset9.12mm
- JP1, JP2: footprint (none) -> Jumper:SolderJumper-2_P1.3mm_Open_TrianglePad1.0x1.5mm
- L1: footprint (none) -> Inductor_SMD:L_6.3x6.3_H3
- R1: renamed from R11; footprint (none) -> Resistor_SMD:R_0603_1608Metric
- R10: renamed from R14; footprint (none) -> Resistor_SMD:R_0603_1608Metric
- R11: renamed from R15; footprint (none) -> Resistor_SMD:R_0603_1608Metric
- R12, R13: footprint (none) -> Resistor_SMD:R_0603_1608Metric
- R14: renamed from R43; footprint (none) -> Resistor_SMD:R_0603_1608Metric
- R15: renamed from R16; footprint (none) -> Resistor_SMD:R_0603_1608Metric
- R16: renamed from R17; footprint (none) -> Resistor_SMD:R_0603_1608Metric
- R17: renamed from R19; footprint (none) -> Resistor_SMD:R_0603_1608Metric
- R18: renamed from R20; footprint (none) -> Resistor_SMD:R_0603_1608Metric
- R19: renamed from R37; footprint (none) -> Resistor_SMD:R_0603_1608Metric
- R2: renamed from R1; footprint (none) -> Resistor_SMD:R_0603_1608Metric
- R20: renamed from R42; footprint (none) -> Resistor_SMD:R_0603_1608Metric
- R21: renamed from R41; footprint (none) -> Resistor_SMD:R_0603_1608Metric
- R22: renamed from R38; footprint (none) -> Resistor_SMD:R_0603_1608Metric
- R23: renamed from R40; footprint (none) -> Resistor_SMD:R_0603_1608Metric
- R24: renamed from R7; footprint (none) -> Resistor_SMD:R_0603_1608Metric
- R25: renamed from R8; footprint (none) -> Resistor_SMD:R_0603_1608Metric
- R26: renamed from R39; footprint (none) -> Resistor_SMD:R_0603_1608Metric
- R27: renamed from R36; footprint (none) -> Resistor_SMD:R_0603_1608Metric
- R28: renamed from R22; footprint (none) -> Resistor_SMD:R_0603_1608Metric
- R29: renamed from R23; footprint (none) -> Resistor_SMD:R_0603_1608Metric
- R3: renamed from R5; footprint (none) -> Resistor_SMD:R_0603_1608Metric
- R30: renamed from R24; footprint (none) -> Resistor_SMD:R_0603_1608Metric
- R31: renamed from R25; footprint (none) -> Resistor_SMD:R_0603_1608Metric
- R32: renamed from R35; footprint (none) -> Resistor_SMD:R_0603_1608Metric
- R33: renamed from R34; footprint (none) -> Resistor_SMD:R_0603_1608Metric
- R34: renamed from R21; footprint (none) -> Resistor_SMD:R_0603_1608Metric
- R35: renamed from R18; footprint (none) -> Resistor_SMD:R_0603_1608Metric
- R36: renamed from R26; footprint (none) -> Resistor_SMD:R_0603_1608Metric
- R37: renamed from R27; footprint (none) -> Resistor_SMD:R_0603_1608Metric
- R38: renamed from R28; footprint (none) -> Resistor_SMD:R_0603_1608Metric
- R39: renamed from R29; footprint (none) -> Resistor_SMD:R_0603_1608Metric
- R4: renamed from R2; footprint (none) -> Resistor_SMD:R_0603_1608Metric
- R40: renamed from R30; footprint (none) -> Resistor_SMD:R_0603_1608Metric
- R41: renamed from R31; footprint (none) -> Resistor_SMD:R_0603_1608Metric
- R42: renamed from R32; footprint (none) -> Resistor_SMD:R_0603_1608Metric
- R5: renamed from R9; footprint (none) -> Resistor_SMD:R_0603_1608Metric
- R6: renamed from R3; footprint (none) -> Resistor_SMD:R_0603_1608Metric
- R7: renamed from R10; footprint (none) -> Resistor_SMD:R_0603_1608Metric
- R8: renamed from R4; footprint (none) -> Resistor_SMD:R_0603_1608Metric
- R9: renamed from R6; footprint (none) -> Resistor_SMD:R_0603_1608Metric
- SW1: renamed from SW2; footprint (none) -> Button_Switch_THT:SW_DIP_SPSTx07_Slide_9.78x19.96mm_W7.62mm_P2.54mm
- U1: renamed from U2; value (none) -> PS/2 Dual port; footprint (none) -> Connector_DIN:PS-2_Dual_Stacked
- U10: footprint (none) -> Package_SO:TSSOP-16_4.4x5mm_P0.65mm
- U2: renamed from U1; footprint (none) -> Module:Tang-Nano-9K
- Y1: footprint (none) -> Crystal:Crystal_SMD_3225-4Pin_3.2x2.5mm
- renumbered D3 to D2, D4 to D3, D2 to D4, U8 to U11, U4 to U3, U5 to U4, U3 to U5, U11 to U7, U9 to U8, U7 to U9
