File: KiCad/tang-nano-9k-shield.kicad_sch (KiCad schematic)
At the start: 104 parts, among them J1 Barrel_Jack, J2 DE15_Socket_HighDensity_Mount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, J3 I2C_headers, J4 AudioJack3, J5 SPI_headers, J6 USB_C_Receptacle_USB2.0_16P, J7 DE9_Socket_MountingHoles, Q1 SS8050, SW1 SW_DIP_x08, U1 PS/2 Dual port, U10 MAX3232, U11 RP2040, U2 Tang Nano 9K, U3 AMS1117-3.3, U4 PT8211, U5 TPS563201DDCR, U6 TPA6132A2RTE, U7 AMS1117-1.8, U8 W25Q32JVZP, U9 USBLC6-2SC6, Y1 X322512MSB4SI

Commit message: Add files via upload
Parts:
- added C34, C35: 100nF, Capacitor_SMD:C_0603_1608Metric, symbol Device:C_Small
- added C36: 1uF, Capacitor_SMD:C_0603_1608Metric, symbol Device:C_Small
- added J8: Pmod, Connector_PinSocket_2.54mm:PinSocket_2x06_P2.54mm_Horizontal, symbol Connector_Generic:Conn_02x06_Odd_Even
- added Q2, Q3, Q4, Q5: BSS138, Package_TO_SOT_SMD:SOT-23, symbol Transistor_FET:BSS138
- added R43, R45, R46, R47, R48, R49, R50, R51, R52: 10K, Resistor_SMD:R_0603_1608Metric, symbol Device:R_Small
- added R44: 180R, Resistor_SMD:R_0603_1608Metric, symbol Device:R_Small
- added R53, R54, R55, R56: 4K7, Resistor_SMD:R_0603_1608Metric, symbol Device:R_Small
- added SW2: SW_DIP_x08, Button_Switch_THT:SW_DIP_SPSTx08_Slide_9.78x22.5mm_W7.62mm_P2.54mm, symbol Switch:SW_DIP_x08
- added U12: TXS0108EPW, Package_SO:TSSOP-20_4.4x6.5mm_P0.65mm, symbol Logic_LevelTranslator:TXS0108EPW
- SW1: footprint Button_Switch_THT:SW_DIP_SPSTx07_Slide_9.78x19.96mm_W7.62mm_P2.54mm -> Button_Switch_THT:SW_DIP_SPSTx08_Slide_9.78x22.5mm_W7.62mm_P2.54mm
Connections:
- net 1V8: now also C34.2, R43.2, R44.1, U12.2 (VCCA); no longer R14.1, R20.1, R21.1, R23.1, R26.1, R27.1, R32.1, R33.1
- net 3V3: now also R14.1, R20.1, R21.1, R23.1, R26.1, R27.1, R32.1, R33.1, C35.1, J8.11 (Pin_11), J8.12 (Pin_12), Q2.1 (G), Q3.1 (G), Q4.1 (G), Q5.1 (G), R45.1, R46.1, R47.1, R48.1, R49.1, R50.1, R51.1, R52.1, R53.1, R54.1, R55.1, R56.1, U12.19 (VCCB); no longer R2.1, R4.1, R6.1, R8.1
- net 5V: now also R2.1, R4.1, R6.1, R8.1
- net GND: now also U11.19 (TESTEN), C34.1, C35.2, C36.1, J8.10 (Pin_10), J8.9 (Pin_9), R44.2, SW2.10, SW2.11, SW2.12, SW2.13, SW2.14, SW2.15, SW2.16, SW2.9, U12.11 (GND)
- net PS/2_CLK1: now also Q2.2 (S), R53.2; no longer R1.2, R2.2
- net PS/2_CLK2: now also Q4.2 (S), R55.2; no longer R5.2, R6.2
- net PS/2_DAT1: now also Q3.2 (S), R54.2; no longer R3.2, R4.2
- net PS/2_DAT2: now also Q5.2 (S), R56.2; no longer R7.2, R8.2
- net SW1: now also U11.2 (GPIO0); no longer U2.86 (IOT8A)
- net SW2: now also U11.3 (GPIO1); no longer U2.85 (IOT8B)
- net SW3: now also U11.4 (GPIO2); no longer U2.84 (IOT10A)
- net SW4: now also U11.5 (GPIO3); no longer U2.83 (IOT10B)
- net SW5: now also U11.6 (GPIO4); no longer U2.82 (IOT11A)
- net SW6: now also U11.7 (GPIO5); no longer U2.81 (IOT11B)
- net SW7: now also U11.8 (GPIO6); no longer U2.80 (IOT12A)
- net SW8: now also U11.9 (GPIO7); no longer U2.79 (IOT12B)
- net SW9: now reaches U11.11 (GPIO8)
- net SW9: now also R52.2, SW2.1
- net SW10: now reaches U11.12 (GPIO9)
- net SW10: now also R51.2, SW2.2
- net SW11: now reaches U11.13 (GPIO10)
- net SW11: now also R50.2, SW2.3
- net SW12: now reaches U11.14 (GPIO11)
- net SW12: now also R49.2, SW2.4
- net SW13: now reaches U11.15 (GPIO12)
- net SW13: now also R48.2, SW2.5
- net SW14: now reaches U11.16 (GPIO13)
- net SW14: now also R47.2, SW2.6
- net SW15: now reaches U11.17 (GPIO14)
- net SW15: now also R46.2, SW2.7
- net SW16: now reaches U11.18 (GPIO15)
- net SW16: now also R45.2, SW2.8
- new net: C36.2, R43.1, U12.10 (OE)
- new net PM1_1V8: U12.1 (A1), U2.86 (IOT8A)
- new net PM2_1V8: U12.3 (A2), U2.85 (IOT8B)
- new net PM3_1V8: U12.4 (A3), U2.84 (IOT10A)
- new net PM4_1V8: U12.5 (A4), U2.83 (IOT10B)
- new net PM5_1V8: U12.6 (A5), U2.82 (IOT11A)
- new net PM6_1V8: U12.7 (A6), U2.81 (IOT11B)
- new net PM7_1V8: U12.8 (A7), U2.80 (IOT12A)
- new net PM8_1V8: U12.9 (A8), U2.79 (IOT12B)
- new net PMOD1: J8.1 (Pin_1), U12.20 (B1)
- new net PMOD10: J8.8 (Pin_8), U12.12 (B8)
- new net PMOD2: J8.3 (Pin_3), U12.18 (B2)
- new net PMOD3: J8.5 (Pin_5), U12.17 (B3)
- new net PMOD4: J8.7 (Pin_7), U12.16 (B4)
- new net PMOD7: J8.2 (Pin_2), U12.15 (B5)
- new net PMOD8: J8.4 (Pin_4), U12.14 (B6)
- new net PMOD9: J8.6 (Pin_6), U12.13 (B7)
- new net PS/2_CLK1_5V: Q2.3 (D), R1.2, R2.2
- new net PS/2_CLK2_5V: Q4.3 (D), R5.2, R6.2
- new net PS/2_DAT1_5V: Q3.3 (D), R3.2, R4.2
- new net PS/2_DAT2_5V: Q5.3 (D), R7.2, R8.2
- no-connect marks 54 -> 37
Other:
- note added: "PMOD"
- note added: "PS/2 level shifter"
- moved on the sheet: R1, R14, R2, R20, R21, R23, R26, R27, R3, R32, R33, R4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
