File: KiCad/tang-nano-9k-shield.kicad_sch (KiCad schematic)
At the start: 128 parts, among them J1 Barrel_Jack, J2 DE15_Socket_HighDensity_Mount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, J3 I2C_headers, J4 AudioJack3, J5 SPI_headers, J6 USB_C_Receptacle_USB2.0_16P, J7 DE9_Socket_MountingHoles, J8 Pmod, Q1 SS8050, Q2 BSS138, Q3 BSS138, Q4 BSS138, Q5 BSS138, SW1 SW_DIP_x08, SW2 SW_DIP_x08, U1 PS/2 Dual port, U10 MAX3232, U11 RP2040, U12 TXS0108EPW, U2 Tang Nano 9K, U3 AMS1117-3.3, U4 PT8211, U5 TPS563201DDCR, U6 TPA6132A2RTE, U7 AMS1117-1.8, U8 W25Q32JVZP, U9 USBLC6-2SC6, Y1 X322512MSB4SI

Commit message: Add files via upload
Parts:
- removed C24, C28, C30, C31, C32: 100nF, Capacitor_SMD:C_0603_1608Metric, symbol Device:C_Small
- removed J7: DE9_Socket_MountingHoles, Connector_Dsub:DSUB-9_Pins_Horizontal_P2.77x2.84mm_EdgePinOffset7.70mm_Housed_MountingHolesOffset9.12mm, symbol Connector:DE9_Socket_MountingHoles
- removed R44: 180R, Resistor_SMD:R_0603_1608Metric, symbol Device:R_Small
- removed U10: MAX3232, Package_SO:TSSOP-16_4.4x5mm_P0.65mm, symbol Interface_UART:MAX3232
- removed U3: AMS1117-3.3, Package_TO_SOT_SMD:SOT-223-3_TabPin2, symbol Regulator_Linear:AMS1117-3.3
- removed U7: AMS1117-1.8, Package_TO_SOT_SMD:SOT-223-3_TabPin2, symbol Regulator_Linear:AMS1117-1.8
- added D5, D6: SS14, Diode_SMD:D_SMA, symbol Diode:SS14
- added R57, R58: 27R, Resistor_SMD:R_0603_1608Metric, symbol Device:R_Small
- added U3: TLV75533PDBV, Package_TO_SOT_SMD:SOT-23-5, symbol Regulator_Linear:TLV75533PDBV
- added U7: TLV75518PDBV, Package_TO_SOT_SMD:SOT-23-5, symbol Regulator_Linear:TLV75518PDBV
- C1, C21: value 100nF -> 1uF
Connections:
- net 1V8: now also U7.5 (OUT)
- net 3V3: now also U3.5 (OUT), U7.1 (IN), U7.3 (EN)
- net 5V: now also D5.1 (K), D6.2 (A), U3.1 (IN), U3.3 (EN); no longer C5.1, U2.5V
- net D1+: now also R58.1; no longer U11.47 (USB_DP)
- net D1-: now also R57.1; no longer U11.46 (USB_DM)
- net GND: now also U3.2 (GND), U7.2 (GND)
- net RS_RX: no longer names the net of U2.70 (IOT41B)
- net RS_TX: no longer names the net of U2.71 (IOT41A)
- new net: R57.2, U11.46 (USB_DM)
- new net: R58.2, U11.47 (USB_DP)
- new net TANG_5V: C5.1, D5.2 (A), D6.1 (K), U2.5V
- no-connect marks 37 -> 29
Other:
- note removed: "RS-232"
- moved on the sheet: C1, C21, D2, D3

Commit message: Add files via upload
Parts:
- removed BZ1: Buzzer, Buzzer_Beeper:MagneticBuzzer_ProSignal_ABT-410-RC, symbol Device:Buzzer
- removed C10, C11: 2.2nF, Capacitor_SMD:C_0603_1608Metric, symbol Device:C_Small
- removed C12, C13, C15, C16, C20, C9: 1uF, Capacitor_SMD:C_0603_1608Metric, symbol Device:C_Small
- removed C18: 2.2uF, Capacitor_SMD:C_0603_1608Metric, symbol Device:C_Small
- removed C8: 100nF, Capacitor_SMD:C_0603_1608Metric, symbol Device:C_Small
- removed D4: 1N4148W, Diode_SMD:D_SOD-123, symbol Diode:1N4148W
- removed J4: AudioJack3, Connector_Audio:Jack_3.5mm_KoreanHropartsElec_PJ-320D-4A_Horizontal, symbol Connector_Audio:AudioJack3
- removed Q1: SS8050, Package_TO_SOT_SMD:SOT-23, symbol Transistor_BJT:SS8050
- removed R12, R13: 47R, Resistor_SMD:R_0603_1608Metric, symbol Device:R_Small
- removed R34: 10K, Resistor_SMD:R_0603_1608Metric, symbol Device:R_Small
- removed R35: 1K, Resistor_SMD:R_0603_1608Metric, symbol Device:R_Small
- removed U4: PT8211, PT8211:SOP8-6.0-4.9X3.9, symbol PT8211:PT8211
- removed U6: TPA6132A2RTE, Package_DFN_QFN:WQFN-16-1EP_3x3mm_P0.5mm_EP1.6x1.6mm_ThermalVias, symbol Amplifier_Audio:TPA6132A2RTE
- added C28, C30, C32, C37, C38, C39, C40: 100nF, Capacitor_SMD:C_0603_1608Metric, symbol Device:C_Small
- added C31: 1uF, Capacitor_SMD:C_0603_1608Metric, symbol Device:C_Small
- added R59, R60: 1K, Resistor_SMD:R_0603_1608Metric, symbol Device:R_Small
- C1, C21, C36: LCSC (none) -> C15849
- C14, C23, C25, C27, C34, C35, C4, C5, C7: LCSC (none) -> C14663
- C17, C19: LCSC (none) -> C12891
- C2, C22, C3, C6: LCSC (none) -> C13585
- C26, C29: value 20pF -> 15pF; LCSC (none) -> C1644
- C33: value 100nF -> 1uF; LCSC (none) -> C15849
- D1, D2, D3, D5, D6: LCSC (none) -> C2480
- J2: footprint Connector_Dsub:DSUB-15-HD_Pins_Horizontal_P2.29x2.54mm_EdgePinOffset8.35mm_Housed_MountingHolesOffset10.89mm -> Connector_Dsub:DSUB-15-HD_Socket_Horizontal_P2.29x2.54mm_EdgePinOffset8.35mm_Housed_MountingHolesOffset10.89mm
- J3: value I2C_headers -> I2C_header; symbol Connector:Conn_01x04_Socket -> Connector_Generic:Conn_01x04
- J6: LCSC (none) -> C2988369
- JP1: value SolderJumper_2_Open -> BOOT
- L1: footprint Inductor_SMD:L_6.3x6.3_H3 -> Inductor_SMD:L_Sunlord_SWPA6045S; LCSC (none) -> C279943; MPN (none) -> SWPA6045S3R3NT; Manufacturer (none) -> Sunlord
- Q2, Q3, Q4, Q5: LCSC (none) -> C7420339
- R1, R3, R5, R7: LCSC (none) -> C23138
- R10, R11: LCSC (none) -> C22775
- R14, R20, R21, R23, R25, R26, R27, R32, R33, R40, R43, R45, R46, R47, R48, R49, R50, R51, R52, R9: LCSC (none) -> C25804
- R15, R28, R36: LCSC (none) -> C23193
- R16, R29, R37: LCSC (none) -> C21190
- R17, R30, R38: LCSC (none) -> C22975
- R18, R31, R39: LCSC (none) -> C23018
- R19, R2, R22, R4, R53, R54, R55, R56, R6, R8: LCSC (none) -> C23162
- R24: value 54K9 -> 56K; LCSC (none) -> C23206
- R41, R42: LCSC (none) -> C23186
- R57, R58: LCSC (none) -> C25190
- U11: LCSC (none) -> C2040
- U12: LCSC (none) -> C17206
- U3: LCSC (none) -> C404027
- U5: LCSC (none) -> C116592
- U7: LCSC (none) -> C2877863
- U8: LCSC (none) -> C571260
- U9: LCSC (none) -> C7519
- Y1: value X322512MSB4SI -> ABM8-272-T3; symbol Device:Crystal_GND23_Small -> Device:Crystal_GND24_Small
Connections:
- net 3V3: now also C28.2, C30.2, C31.2, C32.2, C37.2, C38.2, C39.2, C40.2
- net BOOTSEL: now also R60.2; no longer JP1.2 (B)
- net GND: now also Y1.4 (G), C28.1, C30.1, C31.1, C32.1, C37.1, C38.1, C39.1, C40.1; no longer Y1.3 (G)
- net SCL: now also U11.35 (GPIO23); no longer U2.69 (IOT42A)
- net SDA: now also U11.34 (GPIO22); no longer U2.68 (IOT42B)
- net XOUT: now also Y1.3, R59.1; no longer U11.21 (XOUT), Y1.4
- net TXS_OE: now reaches C36.2, R43.1, U12.10 (OE)
- net BCK: no longer names the net of U2.74 (IOT38B)
- net BUZ: no longer names the net of U2.75 (IOT38A)
- net DIN: no longer names the net of U2.72 (IOT39B)
- net WS: no longer names the net of U2.73 (IOT39A)
- new net: JP1.2 (B), R60.1
- new net: R59.2, U11.21 (XOUT)
- no-connect marks 29 -> 33
Other:
- note removed: "AUDIO"
- moved on the sheet: C1, C14, C17, C19, C2, C21, C22, C23, C25, C26, C27, C29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

Commit message: Add files via upload
Parts:
- added C45: 1uF, Capacitor_SMD:C_0603_1608Metric, symbol Device:C_Small
- added C46: 100nF, Capacitor_SMD:C_0603_1608Metric, symbol Device:C_Small
- added C47: 10uF, Capacitor_SMD:C_1206_3216Metric, symbol Device:C_Small
- added C48, C49: 100nF, Capacitor_SMD:C_0402_1005Metric, symbol Device:C_Small
- added R61: 100K, Resistor_SMD:R_0603_1608Metric, symbol Device:R_Small
- added R62: 15K, Resistor_SMD:R_0603_1608Metric, symbol Device:R_Small
- added R63: 20K, Resistor_SMD:R_0603_1608Metric, symbol Device:R_Small
- added R64: 10K, Resistor_SMD:R_0603_1608Metric, symbol Device:R_Small
- added U13: TPS2065CDBV, Package_TO_SOT_SMD:SOT-23-5, symbol Power_Management:TPS2065CDBV
- C28, C30: footprint Capacitor_SMD:C_0603_1608Metric -> Capacitor_SMD:C_0402_1005Metric; LCSC C14663 -> C1525
- C31, C33: footprint Capacitor_SMD:C_0603_1608Metric -> Capacitor_SMD:C_0402_1005Metric; LCSC C15849 -> C52923
Connections:
- net 3V3: now also R64.2
- net 5V: no longer C27.1, U9.5 (VBUS)
- net 5V_BUCK: now also C45.1, C46.1, U13.5 (IN)
- net 5V_USB: now also C27.1, U9.5 (VBUS), C47.1, R62.1, U13.1 (OUT)
- net D1+: now also U9.1 (I/O1); no longer U9.6 (I/O1)
- net D1-: now also U9.3 (I/O2); no longer U9.4 (I/O2)
- net GND: now also C45.2, C46.2, C47.2, C48.1, C49.1, R61.2, R63.2, U13.2 (GND)
- net GREEN: now also R15.2, R16.2, R17.2, R18.2; no longer R28.2, R29.2, R30.2, R31.2
- net PMOD1: now also U12.16 (B4); no longer U12.20 (B1)
- net PMOD10: now also U12.15 (B5); no longer U12.12 (B8)
- net PMOD2: now also U12.17 (B3); no longer U12.18 (B2)
- net PMOD3: now also U12.18 (B2); no longer U12.17 (B3)
- net PMOD4: now also U12.20 (B1); no longer U12.16 (B4)
- net PMOD7: now also U12.12 (B8); no longer U12.15 (B5)
- net PMOD8: now also U12.13 (B7); no longer U12.14 (B6)
- net PMOD9: now also U12.14 (B6); no longer U12.13 (B7)
- net PS/2_CLK1: now also U2.49 (IOR24A); no longer U2.48 (IOR24B)
- net PS/2_CLK2: now also U2.32 (IOB15B); no longer U2.31 (IOB15A)
- net PS/2_DAT1: now also U2.48 (IOR24B); no longer U2.49 (IOR24A)
- net PS/2_DAT2: now also U2.31 (IOB15A); no longer U2.32 (IOB15B)
- net RAW_D1+: now also U9.6 (I/O1); no longer U9.1 (I/O1)
- net RAW_D1-: now also U9.4 (I/O2); no longer U9.3 (I/O2)
- net RED: now also R28.2, R29.2, R30.2, R31.2; no longer R15.2, R16.2, R17.2, R18.2
- net VGA_G0: now also R18.1, U2.53 (IOR15B); no longer R31.1, U2.56 (IOR14A)
- net VGA_G1: now also R17.1, U2.51 (IOR17B); no longer R30.1, U2.57 (IOR13A)
- net VGA_G2: now also R16.1, U2.42 (IOB41B); no longer R29.1, U2.55 (IOR14B)
- net VGA_G3: now also R15.1, U2.41 (IOB41A); no longer R28.1, U2.54 (IOR15A)
- net VGA_R0: now also R31.1, U2.57 (IOR13A); no longer R18.1, U2.53 (IOR15B)
- net VGA_R1: now also R30.1, U2.56 (IOR14A); no longer R17.1, U2.51 (IOR17B)
- net VGA_R2: now also R29.1, U2.55 (IOR14B); no longer R16.1, U2.42 (IOB41B)
- net VGA_R3: now also R28.1, U2.54 (IOR15A); no longer R15.1, U2.41 (IOB41A)
- net DVDD: now reaches C33.2, U11.23 (DVDD), U11.45 (VREG_VOUT), U11.50 (DVDD)
- net DVDD: now also C48.2, C49.2
- net USB_PWR_EN: now reaches U11.32 (GPIO21)
- net USB_PWR_EN: now also R61.1, U13.4 (EN)
- net VBUS_DET: now reaches U11.36 (GPIO24)
- net VBUS_DET: now also R62.2, R63.1
- net USB_FLT: now reaches U11.37 (GPIO25)
- net USB_FLT: now also R64.1, U13.3 (~{FLT})
- no-connect marks 33 -> 30
Other:
- note added: "BSS138 × 4 · 3V3 ↔ 5V · Tang 48/49, 31/32"
- note added: "DIP SWITCHES"
- note added: "EXTENSION HEADERS"
- note added: "J1 6–17 V → buck 5.07 V → 5V → LDO 3V3 / 1V8"
- note added: "J3 I2C (RP2040) · J5 SPI (FPGA, CS2/INT2)"
- note added: "J6 · CC 5k1 · USBLC6 ESD · 27R → RP2040"
- note added: "PS/2 LEVEL SHIFTER"
- note added: "R-DAC 4 bit × RGB · HS 30 · VS 29 · J2 DE15"
- note added: "RP2040"
- note added: "SW1 + SW2 · 16 switches → RP2040 GPIO0–15"
- note added: "TANG NANO"
- note added: "TPS2065C 5V_BUCK → 5V_USB · EN GPIO21 · FLT GPIO25 · DET GPIO24"
- note added: "TXS0108 1V8 ↔ 3V3 · Tang 79–86"
- note added: "U1 dual PS/2 · 5 V side"
- note added: "U2 Tang Nano 9K · TANG_5V via D5 / D6"
- note added: "USB HOST POWER"
- note added: "W25Q32 flash · 12 MHz · SPI0 slave · I2C1 → J3"
- note removed: "DIP Switches"
- note removed: "Extension headers"
- note removed: "PS/2 level shifter"
- note removed: "RP 2040"
- note removed: "Tang Nano"
- moved on the sheet: C1, C14, C17, C19, C2, C21, C22, C23, C25, C26, C27, C28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

Commit message: Add files via upload
Connections:
- net USB_D-: now reaches R57.2, U11.46 (USB_DM)
- net USB_D+: now reaches R58.2, U11.47 (USB_DP)
Changed lines of the file:
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@@
 	(wire
 		(pts
-			(xy 177.8 114.3) (xy 182.88 114.3)
+			(xy 175.26 118.11) (xy 180.34 118.11)
 		)
 		(stroke
@@
 		)
 	)
+	(label "USB_D-"
+		(at 414.02 106.68 0)
+		(effects
+			(font
+				(size 1.27 1.27)
+			)
+			(justify left bottom)
+		)
+	)
+	(label "USB_D+"
+		(at 414.02 109.22 0)
+		(effects
+			(font
+				(size 1.27 1.27)
+			)
+			(justify left bottom)
+		)
+	)
 	(label "D1+"
 		(at 381 210.82 180)
@@
 	(global_label "5V"
 		(shape input)
-		(at 182.88 114.3 0)
+		(at 180.34 118.11 0)
 		(fields_autoplaced yes)
 		(effects
@@
 		)
 		(property "Intersheetrefs" "${INTERSHEET_REFS}"
-			(at 182.88 114.3 0)
+			(at 180.34 118.11 0)
 			(hide yes)
 			(show_name no)
@@
 	(global_label "GND"
 		(shape input)
-		(at 308.61 134.62 0)
+		(at 293.37 134.62 270)
 		(effects
 			(font
 				(size 1.27 1.27)
 			)
-			(justify left)
+			(justify right)
 		)
 		(property "Intersheetrefs" "${INTERSHEET_REFS}"
-			(at 308.61 134.62 0)
+			(at 293.37 134.62 90)
 			(hide yes)
 			(show_name no)
@@
 	(symbol
 		(lib_id "power:PWR_FLAG")
-		(at 177.8 114.3 0)
+		(at 175.26 118.11 0)
 		(unit 1)
 		(body_style 1)
@@
 		(dnp no)
 		(property "Reference" "#FLG0901"
-			(at 177.8 112.39 0)
+			(at 175.26 116.2 0)
 			(hide yes)
 			(show_name no)
@@
 		)
 		(property "Value" "PWR_FLAG"
-			(at 177.8 109.22 0)
+			(at 175.26 113.03 0)
 			(show_name no)
 			(do_not_autoplace no)
@@
 		)
 		(property "Footprint" ""
-			(at 177.8 114.3 0)
+			(at 175.26 118.11 0)
 			(hide yes)
 			(show_name no)
@@
 		)
 		(property "Datasheet" ""
-			(at 177.8 114.3 0)
+			(at 175.26 118.11 0)
 			(hide yes)
 			(show_name no)
@@
 		)
 		(property "Description" "Special symbol for telling ERC where power comes from"
-			(at 177.8 114.3 0)
+			(at 175.26 118.11 0)
 			(hide yes)
 			(show_name no)

Commit message: Add files via upload
Changed lines of the file:
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@@
 	)
 	(junction
+		(at 293.37 134.62)
+		(diameter 0)
+		(color 0 0 0 0)
+	)
+	(junction
 		(at 439.42 53.34)
 		(diameter 0)
@@
 	(wire
 		(pts
+			(xy 293.37 134.62) (xy 302.26 134.62)
+		)
+		(stroke
+			(width 0)
+			(type default)
+		)
+	)
+	(wire
+		(pts
 			(xy 266.7 201.93) (xy 266.7 212.09)
 		)
@@
 	(wire
 		(pts
-			(xy 285.75 134.62) (xy 302.26 134.62)
+			(xy 285.75 134.62) (xy 293.37 134.62)
 		)
 		(stroke
@@
 	(wire
 		(pts
+			(xy 293.37 142.24) (xy 293.37 134.62)
+		)
+		(stroke
+			(width 0)
+			(type default)
+		)
+	)
+	(wire
+		(pts
 			(xy 414.02 238.76) (xy 414.02 241.3)
 		)
@@
 		)
 	)
-	(label "USB_D-"
-		(at 414.02 106.68 0)
-		(effects
-			(font
-				(size 1.27 1.27)
-			)
-			(justify left bottom)
-		)
-	)
-	(label "USB_D+"
-		(at 414.02 109.22 0)
-		(effects
-			(font
-				(size 1.27 1.27)
-			)
-			(justify left bottom)
-		)
-	)
 	(label "D1+"
 		(at 381 210.82 180)
@@
 		)
 	)
+	(label "USB_D+"
+		(at 414.02 109.22 0)
+		(effects
+			(font
+				(size 1.27 1.27)
+			)
+			(justify left bottom)
+		)
+	)
 	(label "CS2"
 		(at 226.06 323.85 180)
@@
 		)
 	)
+	(label "GND"
+		(at 293.37 138.43 180)
+		(effects
+			(font
+				(size 1.27 1.27)
+			)
+			(justify right bottom)
+		)
+	)
 	(label "VGA_B2"
 		(at 393.7 320.04 180)
@@
 		)
 	)
+	(label "USB_D-"
+		(at 414.02 106.68 0)
+		(effects
+			(font
+				(size 1.27 1.27)
+			)
+			(justify left bottom)
+		)
+	)
 	(label "D1+"
 		(at 403.86 109.22 180)
@@
 	(global_label "GND"
 		(shape input)
-		(at 293.37 134.62 270)
+		(at 293.37 142.24 180)
 		(effects
 			(font
@@
 		)
 		(property "Intersheetrefs" "${INTERSHEET_REFS}"
-			(at 293.37 134.62 90)
+			(at 293.37 142.24 0)
 			(hide yes)
 			(show_name no)
