File: KiCad/block_diagram.kicad_sch (KiCad schematic)
At the start: 0 parts

Commit message: Add files via upload
Other:
- note added: "AUDIO AMP"
Changed lines of the file:
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@@
 	)
 	(rectangle
-		(start 230.124 51.562)
-		(end 248.412 69.85)
+		(start 256.794 49.276)
+		(end 275.082 67.564)
 		(stroke
 			(width 0.508)
@@
 	)
 	(rectangle
+		(start 230.124 56.134)
+		(end 252.73 67.564)
+		(stroke
+			(width 0.508)
+			(type solid)
+			(color 0 194 194 1)
+		)
+		(fill
+			(type none)
+		)
+	)
+	(rectangle
 		(start 80.01 57.404)
 		(end 97.282 76.962)
@@
 	)
 	(rectangle
-		(start 203.2 58.166)
-		(end 223.52 69.596)
+		(start 203.2 56.134)
+		(end 223.52 67.564)
 		(stroke
 			(width 0.508)
@@
 	(text "GND\n"
 		(exclude_from_sim no)
-		(at 254.254 66.802 0)
+		(at 280.924 64.516 0)
 		(effects
 			(font
@@
 		)
 	)
+	(text "5V\n"
+		(exclude_from_sim no)
+		(at 244.856 50.292 0)
+		(effects
+			(font
+				(size 2.54 2.54)
+				(thickness 0.508)
+				(bold yes)
+				(color 221 133 0 1)
+			)
+		)
+	)
 	(text "UART\nHeaders"
 		(exclude_from_sim no)
@@
 	(text "I2S DAC"
 		(exclude_from_sim no)
-		(at 213.36 64.008 0)
+		(at 213.36 61.976 0)
 		(effects
 			(font
@@
 	(text "GND\n"
 		(exclude_from_sim no)
-		(at 247.142 89.916 0)
+		(at 246.888 89.662 0)
 		(effects
 			(font
@@
 		)
 	)
-	(text "3V3"
+	(text "5V\n"
 		(exclude_from_sim no)
-		(at 213.614 50.038 0)
+		(at 213.614 48.006 0)
 		(effects
 			(font
@@
 		)
 	)
+	(text "AUDIO AMP\n"
+		(exclude_from_sim no)
+		(at 241.808 62.23 0)
+		(effects
+			(font
+				(size 2.54 2.54)
+				(thickness 0.508)
+				(bold yes)
+				(color 0 194 194 1)
+			)
+		)
+	)
 	(text "5V\n"
 		(exclude_from_sim no)
@@
 	(text "GND\n"
 		(exclude_from_sim no)
-		(at 213.36 76.454 0)
+		(at 213.36 74.422 0)
+		(effects
+			(font
+				(size 2.54 2.54)
+				(thickness 0.508)
+				(bold yes)
+				(color 221 133 0 1)
+			)
+		)
+	)
+	(text "GND\n"
+		(exclude_from_sim no)
+		(at 256.54 71.882 0)
 		(effects
 			(font
@@
 	(polyline
 		(pts
-			(xy 202.692 67.056) (xy 197.866 67.056)
+			(xy 202.692 65.024) (xy 197.866 65.024)
 		)
 		(stroke
@@
 	(polyline
 		(pts
-			(xy 248.412 60.198) (xy 254 60.198)
+			(xy 275.082 57.912) (xy 280.67 57.912)
 		)
 		(stroke
@@
 	(polyline
 		(pts
+			(xy 256.54 65.024) (xy 252.984 65.024)
+		)
+		(stroke
+			(width 0.508)
+			(type solid)
+			(color 0 194 0 1)
+		)
+	)
+	(polyline
+		(pts
 			(xy 236.474 76.454) (xy 242.062 76.454)
 		)
@@
 	(polyline
 		(pts
-			(xy 229.616 67.056) (xy 223.774 67.056)
+			(xy 229.616 65.024) (xy 223.774 65.024)
 		)
 		(stroke
@@
 	(polyline
 		(pts
+			(xy 248.666 71.628) (xy 252.222 71.628)
+		)
+		(stroke
+			(width 0.508)
+			(type solid)
+			(color 221 133 0 1)
+		)
+	)
+	(polyline
+		(pts
 			(xy 146.05 84.074) (xy 141.224 84.074)
 		)
@@
 	(polyline
 		(pts
-			(xy 254.254 63.754) (xy 254.254 60.198)
+			(xy 280.924 61.468) (xy 280.924 57.912)
 		)
 		(stroke
@@
 	(polyline
 		(pts
-			(xy 213.36 69.85) (xy 213.36 73.914)
+			(xy 213.36 67.818) (xy 213.36 71.882)
 		)
 		(stroke
@@
 	(polyline
 		(pts
-			(xy 213.36 52.07) (xy 213.36 57.658)
+			(xy 248.666 71.628) (xy 248.666 67.818)
+		)
+		(stroke
+			(width 0.508)
+			(type solid)
+			(color 221 133 0 1)
+		)
+	)
+	(polyline
+		(pts
+			(xy 213.36 50.038) (xy 213.36 55.626)
 		)
 		(stroke
@@
 		)
 	)
+	(polyline
+		(pts
+			(xy 245.11 55.88) (xy 245.11 52.07)
+		)
+		(stroke
+			(width 0.508)
+			(type solid)
+			(color 221 133 0 1)
+		)
+	)
 	(image
 		(at 229.616 100.584)
@@
 	)
 	(image
-		(at 239.268 60.706)
+		(at 265.938 58.42)
 		(scale 0.474563)
 		(data "/9j/4AAQSkZJRgABAQAAAQABAAD/2wCEAAkGBwgHBgkIBwgKCgkLDRYPDQwMDRsUFRAWIB0iIiAd"

Commit message: Add files via upload
Other:
- note removed: "USB-to-SPI Bridge"

Commit message: Add files via upload
Other:
- note removed: "UART Headers"

Commit message: Add files via upload
Other:
- note added: "12 MHz ABM8"
- note added: "16 × switch"
- note added: "1V8"
- note added: "1V8 LOADS"
- note added: "1V8 ↔ 3V3"
- note added: "2 × 6, 8 I/O"
- note added: "3V3 LOADS"
- note added: "3V3 · SDA · SCL"
- note added: "3V3 ↔ 5V"
- note added: "4 bit × RGB"
- note added: "4.0 – 5 V"
- note added: "5 V"
- note added: "5.07 V"
- note added: "500 mA max"
- note added: "5V · 3V3 · 1V8"
- note added: "5V ≈ 4.6 V"
- note added: "5V_BUCK"
- note added: "5V_USB"
- note added: "6 – 17 V"
- note added: "B [33 34 40 35] · G [41 42 51 53] · R [54–57] · HS [30] · VS [29]"
- note added: "BLOCK DIAGRAM"
- note added: "BSS138 × 4"
- note added: "CS2 [27] INT2 [28]"
- note added: "D+/D− → USBLC6 → 27R → RP2040"
- note added: "D1"
- note added: "D2"
- note added: "D3"
- note added: "D5"
- note added: "D5: Tang → shield · D6: shield → Tang"
- note added: "D6"
- note added: "DE15 female"
- note added: "Dx = Schottky OR-ing, no back-feed"
- note added: "EN = GPIO21"
- note added: "ESD"
- note added: "GPIO"
- note added: "GPIO0–15"
- note added: "GPIO21 / 24 / 25"
- note added: "GW1NR-9 FPGA"
- note added: "HDMI 68–75 unused · SD slot shares SPI (CS 38)"
- note added: "I2C"
- note added: "I2C1 · GPIO22/23"
- note added: "J1 BARREL"
- note added: "J1 barrel 6–17 V"
- note added: "J2 VGA"
- note added: "J3 I2C"
- note added: "J3 · J5 · J8, pull-ups"
- note added: "J5 SPI"
- note added: "J6 USB-C"
- note added: "J8 Pmod"
- note added: "P1 DAT [48] CLK [49] · P2 DAT [31] CLK [32]"
- note added: "POWER TREE"
- note added: "PS/2"
- note added: "PS/2 5 V side"
- note added: "Pmod"
- note added: "R-DAC"
- note added: "RGB444 + sync"
- note added: "RP2040"
- note added: "RP2040 + flash"
- note added: "SPI"
- note added: "SPI · FPGA master"
- note added: "SW1 + SW2 DIP"
- note added: "TANG NANO 9K"
- note added: "TANG USB"
- note added: "TANG_5V"
- note added: "TLV75518"
- note added: "TLV75533"
- note added: "TPS563201"
- note added: "TXS0108"
- note added: "TXS0108 VCCA"
- note added: "TXS0108 VCCB, BSS138"
- note added: "Tang [79–86] (1.8 V bank)"
- note added: "U1 PS/2 × 2"
- note added: "U1, pull-ups"
- note added: "U13 TPS2065C"
- note added: "U13 VBUS switch"
- note added: "U3 LDO"
- note added: "U5 BUCK"
- note added: "U7 LDO"
- note added: "USB"
- note added: "USB FS"
- note added: "USB-C · Tang USB"
- note added: "USBLC6"
- note added: "VBUS"
- note added: "VBUS 5 V"
- note added: "VBUS out"
- note added: "VGA"
- note added: "VIN 2.5 – 5.5 V"
- note added: "VIN 6–17 V"
- note added: "W25Q32 flash"
- note added: "[36/37/39] CS1 [25] INT1 [26]"
- note added: "banks 3.3 V / 1.8 V"
- note added: "centre +"
- note added: "control / VBUS"
- note added: "flash (device)"
- note added: "flash: VBUS in ⇄ USB host: VBUS out"
- note added: "keyboard (host)"
- note added: "keyboard + mouse"
- note added: "load switch 1.5 A"
- note added: "on-board PMU → 3.3 / 1.8 / 1.2 V"
- note added: "power flows left → right · colour = rail · graphics only"
- note added: "protect"
- note added: "see POWER TREE ↓"
- note added: "signal flow · colour = interface · Tang pin numbers in brackets"
- note added: "→ 5.07 V / 3 A"
- note added: "↔ bidirectional · → one way"
- note removed: "AUDIO AMP"
- note removed: "Buck"
- note removed: "Connector"
- note removed: "Electromechanical"
- note removed: "GND"
- note removed: "I2C Headers"
- note removed: "I2S DAC"
- note removed: "IC"
- note removed: "LDO-3.3"
- note removed: "RS-232 Driver"
- note removed: "SIGNAL"
- note removed: "SPI Headers"
