File: KiCad/tang-nano-9k-shield.kicad_pcb (KiCad board)
At the start: 2 copper layers, 104 parts, among them J1 Barrel_Jack, J2 DE15_Socket_HighDensity_Mount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, J3 I2C_headers, J4 AudioJack3, J5 SPI_headers, J6 USB_C_Receptacle_USB2.0_16P, J7 DE9_Socket_MountingHoles, Q1 SS8050, SW1 SW_DIP_x08, U1 PS/2 Dual port, U10 MAX3232, U11 RP2040, U2 Tang Nano 9K, U3 AMS1117-3.3, U4 PT8211, U5 TPS563201DDCR, U6 TPA6132A2RTE, U7 AMS1117-1.8, U8 W25Q32JVZP, U9 USBLC6-2SC6, Y1 X322512MSB4SI

Commit message: Add files via upload
Parts:
- removed BZ1: Buzzer, Buzzer_Beeper:MagneticBuzzer_ProSignal_ABT-410-RC
- removed C10, C11: 2.2nF, Capacitor_SMD:C_0603_1608Metric
- removed C12, C13, C15, C16, C20, C9: 1uF, Capacitor_SMD:C_0603_1608Metric
- removed C18: 2.2uF, Capacitor_SMD:C_0603_1608Metric
- removed C24, C8: 100nF, Capacitor_SMD:C_0603_1608Metric
- removed D4: 1N4148W, Diode_SMD:D_SOD-123
- removed J4: AudioJack3, Connector_Audio:Jack_3.5mm_KoreanHropartsElec_PJ-320D-4A_Horizontal
- removed J7: DE9_Socket_MountingHoles, Connector_Dsub:DSUB-9_Pins_Horizontal_P2.77x2.84mm_EdgePinOffset7.70mm_Housed_MountingHolesOffset9.12mm
- removed Q1: SS8050, Package_TO_SOT_SMD:SOT-23
- removed R12, R13: 47R, Resistor_SMD:R_0603_1608Metric
- removed R34: 10K, Resistor_SMD:R_0603_1608Metric
- removed R35: 1K, Resistor_SMD:R_0603_1608Metric
- removed U10: MAX3232, Package_SO:TSSOP-16_4.4x5mm_P0.65mm
- removed U4: PT8211, PT8211:SOP8-6.0-4.9X3.9
- removed U6: TPA6132A2RTE, Package_DFN_QFN:WQFN-16-1EP_3x3mm_P0.5mm_EP1.6x1.6mm_ThermalVias
- added C34: 100nF, Capacitor_SMD:C_0603_1608Metric, F.Cu at (164.4, 84.5)
- added C35: 100nF, Capacitor_SMD:C_0603_1608Metric, F.Cu at (164.4, 87.0)
- added C36: 1uF, Capacitor_SMD:C_0603_1608Metric, F.Cu at (164.4, 89.5)
- added C37: 100nF, Capacitor_SMD:C_0603_1608Metric, F.Cu at (164.4, 92.0)
- added C38: 100nF, Capacitor_SMD:C_0603_1608Metric, F.Cu at (164.4, 94.5)
- added C39: 100nF, Capacitor_SMD:C_0603_1608Metric, F.Cu at (164.4, 97.0)
- added C40: 100nF, Capacitor_SMD:C_0603_1608Metric, F.Cu at (164.4, 99.6)
- added D5: SS14, Diode_SMD:D_SMA, F.Cu at (146.3, 115.8)
- added D6: SS14, Diode_SMD:D_SMA, F.Cu at (146.3, 120.3)
- added J8: Pmod, Connector_PinSocket_2.54mm:PinSocket_2x06_P2.54mm_Horizontal, F.Cu at (172.0, 110.6)
- added Q2: BSS138, Package_TO_SOT_SMD:SOT-23, F.Cu at (176.8, 110.6)
- added Q3: BSS138, Package_TO_SOT_SMD:SOT-23, F.Cu at (176.8, 115.0)
- added Q4: BSS138, Package_TO_SOT_SMD:SOT-23, F.Cu at (176.8, 119.5)
- added Q5: BSS138, Package_TO_SOT_SMD:SOT-23, F.Cu at (176.8, 123.9)
- added R43: 10K, Resistor_SMD:R_0603_1608Metric, F.Cu at (176.4, 99.6)
- added R45: 10K, Resistor_SMD:R_0603_1608Metric, F.Cu at (176.4, 102.1)
- added R46: 10K, Resistor_SMD:R_0603_1608Metric, F.Cu at (176.4, 104.6)
- added R47: 10K, Resistor_SMD:R_0603_1608Metric, F.Cu at (176.4, 107.1)
- added R48: 10K, Resistor_SMD:R_0603_1608Metric, F.Cu at (180.4, 77.0)
- added R49: 10K, Resistor_SMD:R_0603_1608Metric, F.Cu at (180.4, 79.5)
- added R50: 10K, Resistor_SMD:R_0603_1608Metric, F.Cu at (180.4, 82.0)
- added R51: 10K, Resistor_SMD:R_0603_1608Metric, F.Cu at (180.4, 84.5)
- added R52: 10K, Resistor_SMD:R_0603_1608Metric, F.Cu at (180.4, 87.0)
- added R53: 4K7, Resistor_SMD:R_0603_1608Metric, F.Cu at (180.4, 89.5)
- added R54: 4K7, Resistor_SMD:R_0603_1608Metric, F.Cu at (180.4, 92.0)
- added R55: 4K7, Resistor_SMD:R_0603_1608Metric, F.Cu at (180.4, 94.5)
- added R56: 4K7, Resistor_SMD:R_0603_1608Metric, F.Cu at (180.4, 97.0)
- added R57: 27R, Resistor_SMD:R_0603_1608Metric, F.Cu at (180.4, 99.6)
- added R58: 27R, Resistor_SMD:R_0603_1608Metric, F.Cu at (180.4, 102.1)
- added R59: 1K, Resistor_SMD:R_0603_1608Metric, F.Cu at (180.4, 104.6)
- added R60: 1K, Resistor_SMD:R_0603_1608Metric, F.Cu at (180.4, 107.1)
- added SW2: SW_DIP_x08, Button_Switch_THT:SW_DIP_SPSTx08_Slide_9.78x22.5mm_W7.62mm_P2.54mm, F.Cu at (195.8, 78.9)
- added U12: TXS0108EPW, Package_SO:TSSOP-20_4.4x6.5mm_P0.65mm, F.Cu at (192.5, 62.3)
- C1, C21, C31, C33: value 100nF -> 1uF
- C26, C29: value 20pF -> 15pF
- J2: footprint Connector_Dsub:DSUB-15-HD_Pins_Horizontal_P2.29x2.54mm_EdgePinOffset8.35mm_Housed_MountingHolesOffset10.89mm -> Connector_Dsub:DSUB-15-HD_Socket_Horizontal_P2.29x2.54mm_EdgePinOffset8.35mm_Housed_MountingHolesOffset10.89mm
- J3: value I2C_headers -> I2C_header
- JP1: value SolderJumper_2_Open -> BOOT
- L1: footprint Inductor_SMD:L_6.3x6.3_H3 -> Inductor_SMD:L_Sunlord_SWPA6045S
- R24: value 54K9 -> 56K
- SW1: footprint Button_Switch_THT:SW_DIP_SPSTx07_Slide_9.78x19.96mm_W7.62mm_P2.54mm -> Button_Switch_THT:SW_DIP_SPSTx08_Slide_9.78x22.5mm_W7.62mm_P2.54mm
- U3: value AMS1117-3.3 -> TLV75533PDBV; footprint Package_TO_SOT_SMD:SOT-223-3_TabPin2 -> Package_TO_SOT_SMD:SOT-23-5
- U7: value AMS1117-1.8 -> TLV75518PDBV; footprint Package_TO_SOT_SMD:SOT-223-3_TabPin2 -> Package_TO_SOT_SMD:SOT-23-5
- Y1: value X322512MSB4SI -> ABM8-272-T3
- moved L1 106.3 mm to (191.7, 70.1)
- moved J5 104.9 mm to (203.0, 102.2)
- moved R32 99.9 mm to (176.4, 77.0)
- moved R33 99.9 mm to (176.4, 79.5)
- moved R19 98.7 mm to (172.4, 77.0)
- moved R20 98.7 mm to (172.4, 79.5)
- moved R21 98.7 mm to (172.4, 82.0)
- moved U8 97.1 mm to (201.7, 52.3)
- moved C14 95.3 mm to (160.4, 87.0)
- moved R4 95.3 mm to (168.4, 77.0)
- moved R5 95.3 mm to (168.4, 79.5)
- moved R6 95.3 mm to (168.4, 82.0)
- moved R7 95.3 mm to (168.4, 84.5)
- moved R8 95.3 mm to (168.4, 87.0)
- moved R9 95.3 mm to (168.4, 89.5)
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Connections:
- C30 pad 1: Net-(U10-C2+) -> GND
- C30 pad 2: Net-(U10-C2-) -> 3V3
- C31 pad 1: Net-(U10-VS+) -> GND
- C31 pad 2: GND -> 3V3
- C32 pad 1: Net-(U10-VS-) -> GND
- C32 pad 2: GND -> 3V3
- C5 pad 1: 5V -> /tang-nano-9k-shield/TANG_5V
- JP1 pad 2: /tang-nano-9k-shield/BOOTSEL -> Net-(JP1-B)
- R1 pad 2: /tang-nano-9k-shield/PS/2_CLK1 -> /tang-nano-9k-shield/PS/2_CLK1_5V
- R14 pad 1: 1V8 -> 3V3
- R2 pad 1: 3V3 -> 5V
- R2 pad 2: /tang-nano-9k-shield/PS/2_CLK1 -> /tang-nano-9k-shield/PS/2_CLK1_5V
- R20 pad 1: 1V8 -> 3V3
- R21 pad 1: 1V8 -> 3V3
- R23 pad 1: 1V8 -> 3V3
- R26 pad 1: 1V8 -> 3V3
- R27 pad 1: 1V8 -> 3V3
- R3 pad 2: /tang-nano-9k-shield/PS/2_DAT1 -> /tang-nano-9k-shield/PS/2_DAT1_5V
- R32 pad 1: 1V8 -> 3V3
- R33 pad 1: 1V8 -> 3V3
- R4 pad 1: 3V3 -> 5V
- R4 pad 2: /tang-nano-9k-shield/PS/2_DAT1 -> /tang-nano-9k-shield/PS/2_DAT1_5V
- R5 pad 2: /tang-nano-9k-shield/PS/2_CLK2 -> /tang-nano-9k-shield/PS/2_CLK2_5V
- R6 pad 1: 3V3 -> 5V
- R6 pad 2: /tang-nano-9k-shield/PS/2_CLK2 -> /tang-nano-9k-shield/PS/2_CLK2_5V
- R7 pad 2: /tang-nano-9k-shield/PS/2_DAT2 -> /tang-nano-9k-shield/PS/2_DAT2_5V
- R8 pad 1: 3V3 -> 5V
- R8 pad 2: /tang-nano-9k-shield/PS/2_DAT2 -> /tang-nano-9k-shield/PS/2_DAT2_5V
- U11 pad 11: unconnected-(U11-GPIO8-Pad11) -> /tang-nano-9k-shield/SW9
- U11 pad 12: unconnected-(U11-GPIO9-Pad12) -> /tang-nano-9k-shield/SW10
- U11 pad 13: unconnected-(U11-GPIO10-Pad13) -> /tang-nano-9k-shield/SW11
- U11 pad 14: unconnected-(U11-GPIO11-Pad14) -> /tang-nano-9k-shield/SW12
- U11 pad 15: unconnected-(U11-GPIO12-Pad15) -> /tang-nano-9k-shield/SW13
- U11 pad 16: unconnected-(U11-GPIO13-Pad16) -> /tang-nano-9k-shield/SW14
- U11 pad 17: unconnected-(U11-GPIO14-Pad17) -> /tang-nano-9k-shield/SW15
- U11 pad 18: unconnected-(U11-GPIO15-Pad18) -> /tang-nano-9k-shield/SW16
- U11 pad 19: unconnected-(U11-TESTEN-Pad19) -> GND
- U11 pad 2: unconnected-(U11-GPIO0-Pad2) -> /tang-nano-9k-shield/SW1
- U11 pad 21: /tang-nano-9k-shield/XOUT -> Net-(U11-XOUT)
- U11 pad 3: unconnected-(U11-GPIO1-Pad3) -> /tang-nano-9k-shield/SW2
- U11 pad 34: unconnected-(U11-GPIO22-Pad34) -> /tang-nano-9k-shield/SDA
- U11 pad 35: unconnected-(U11-GPIO23-Pad35) -> /tang-nano-9k-shield/SCL
- U11 pad 4: unconnected-(U11-GPIO2-Pad4) -> /tang-nano-9k-shield/SW3
- U11 pad 46: /tang-nano-9k-shield/D1- -> Net-(U11-USB_DM)
- U11 pad 47: /tang-nano-9k-shield/D1+ -> Net-(U11-USB_DP)
- U11 pad 5: unconnected-(U11-GPIO3-Pad5) -> /tang-nano-9k-shield/SW4
- U11 pad 6: unconnected-(U11-GPIO4-Pad6) -> /tang-nano-9k-shield/SW5
- U11 pad 7: unconnected-(U11-GPIO5-Pad7) -> /tang-nano-9k-shield/SW6
- U11 pad 8: unconnected-(U11-GPIO6-Pad8) -> /tang-nano-9k-shield/SW7
- U11 pad 9: unconnected-(U11-GPIO7-Pad9) -> /tang-nano-9k-shield/SW8
- U2 pad 5V: 5V -> /tang-nano-9k-shield/TANG_5V
- U2 pad 68: /tang-nano-9k-shield/SDA -> unconnected-(U2-IOT42B-Pad68)
- U2 pad 69: /tang-nano-9k-shield/SCL -> unconnected-(U2-IOT42A-Pad69)
- U2 pad 70: /tang-nano-9k-shield/RS_RX -> unconnected-(U2-IOT41B-Pad70)
- U2 pad 71: /tang-nano-9k-shield/RS_TX -> unconnected-(U2-IOT41A-Pad71)
- U2 pad 72: /tang-nano-9k-shield/DIN -> unconnected-(U2-IOT39B-Pad72)
- U2 pad 73: /tang-nano-9k-shield/WS -> unconnected-(U2-IOT39A-Pad73)
- U2 pad 74: /tang-nano-9k-shield/BCK -> unconnected-(U2-IOT38B-Pad74)
- U2 pad 75: /tang-nano-9k-shield/BUZ -> unconnected-(U2-IOT38A-Pad75)
- U2 pad 79: /tang-nano-9k-shield/SW8 -> /tang-nano-9k-shield/PM8_1V8
- U2 pad 80: /tang-nano-9k-shield/SW7 -> /tang-nano-9k-shield/PM7_1V8
- U2 pad 81: /tang-nano-9k-shield/SW6 -> /tang-nano-9k-shield/PM6_1V8
- U2 pad 82: /tang-nano-9k-shield/SW5 -> /tang-nano-9k-shield/PM5_1V8
- U2 pad 83: /tang-nano-9k-shield/SW4 -> /tang-nano-9k-shield/PM4_1V8
- U2 pad 84: /tang-nano-9k-shield/SW3 -> /tang-nano-9k-shield/PM3_1V8
- U2 pad 85: /tang-nano-9k-shield/SW2 -> /tang-nano-9k-shield/PM2_1V8
- U2 pad 86: /tang-nano-9k-shield/SW1 -> /tang-nano-9k-shield/PM1_1V8
- U3 pad 1: GND -> 5V
- U3 pad 2: 3V3 -> GND
- U7 pad 1: GND -> 3V3
- U7 pad 2: 1V8 -> GND
- Y1 pad 3: GND -> /tang-nano-9k-shield/XOUT
- Y1 pad 4: /tang-nano-9k-shield/XOUT -> GND

Commit message: Add files via upload
Parts:
- added C45: 1uF, Capacitor_SMD:C_0603_1608Metric, F.Cu at (176.7, 145.5)
- added C46: 100nF, Capacitor_SMD:C_0603_1608Metric, F.Cu at (178.2, 145.5)
- added C47: 10uF, Capacitor_SMD:C_1206_3216Metric, F.Cu at (177.1, 153.7)
- added C48: 100nF, Capacitor_SMD:C_0402_1005Metric, F.Cu at (171.0, 141.8)
- added C49: 100nF, Capacitor_SMD:C_0402_1005Metric, F.Cu at (169.0, 131.6)
- added R61: 100K, Resistor_SMD:R_0603_1608Metric, F.Cu at (180.1, 145.5)
- added R62: 15K, Resistor_SMD:R_0603_1608Metric, F.Cu at (175.2, 153.1)
- added R63: 20K, Resistor_SMD:R_0603_1608Metric, F.Cu at (175.2, 156.1)
- added R64: 10K, Resistor_SMD:R_0603_1608Metric, F.Cu at (180.5, 152.9)
- added U13: TPS2065CDBV, Package_TO_SOT_SMD:SOT-23-5, F.Cu at (179.2, 149.2)
- C28, C30, C31, C33: footprint Capacitor_SMD:C_0603_1608Metric -> Capacitor_SMD:C_0402_1005Metric
- moved R36 145.5 mm to (40.8, 134.7), turned to 180 degrees
- moved R37 145.2 mm to (40.8, 136.3), turned to 180 degrees
- moved R38 144.9 mm to (40.8, 137.9), turned to 180 degrees
- moved R39 144.5 mm to (40.8, 139.5), turned to 180 degrees
- moved R28 141.7 mm to (40.8, 152.1), turned to 180 degrees
- moved R29 141.4 mm to (40.8, 153.7), turned to 180 degrees
- moved R30 141.0 mm to (40.8, 155.3), turned to 180 degrees
- moved R31 140.7 mm to (40.8, 156.8), turned to 180 degrees
- moved J2 137.4 mm to (27.3, 147.8), turned to -90 degrees
- moved R15 135.0 mm to (40.8, 143.5), turned to 180 degrees
- moved R16 134.6 mm to (40.8, 145.0), turned to 180 degrees
- moved R17 134.3 mm to (40.8, 146.6), turned to 180 degrees
- moved R18 134.1 mm to (40.8, 148.1), turned to 180 degrees
- moved R10 133.5 mm to (40.8, 131.1)
- moved R11 131.8 mm to (40.9, 127.9)
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Connections:
- net /tang-nano-9k-shield/BLUE renamed BLUE
- net Net-(U11-VREG_VOUT) renamed /tang-nano-9k-shield/DVDD
- C27 pad 1: 5V -> 5V_USB
- J2 pad 1: /tang-nano-9k-shield/RED -> RED
- J2 pad 2: /tang-nano-9k-shield/GREEN -> GREEN
- R15 pad 1: /tang-nano-9k-shield/VGA_R3 -> /tang-nano-9k-shield/VGA_G3
- R15 pad 2: /tang-nano-9k-shield/RED -> GREEN
- R16 pad 1: /tang-nano-9k-shield/VGA_R2 -> /tang-nano-9k-shield/VGA_G2
- R16 pad 2: /tang-nano-9k-shield/RED -> GREEN
- R17 pad 1: /tang-nano-9k-shield/VGA_R1 -> /tang-nano-9k-shield/VGA_G1
- R17 pad 2: /tang-nano-9k-shield/RED -> GREEN
- R18 pad 1: /tang-nano-9k-shield/VGA_R0 -> /tang-nano-9k-shield/VGA_G0
- R18 pad 2: /tang-nano-9k-shield/RED -> GREEN
- R28 pad 1: /tang-nano-9k-shield/VGA_G3 -> /tang-nano-9k-shield/VGA_R3
- R28 pad 2: /tang-nano-9k-shield/GREEN -> RED
- R29 pad 1: /tang-nano-9k-shield/VGA_G2 -> /tang-nano-9k-shield/VGA_R2
- R29 pad 2: /tang-nano-9k-shield/GREEN -> RED
- R30 pad 1: /tang-nano-9k-shield/VGA_G1 -> /tang-nano-9k-shield/VGA_R1
- R30 pad 2: /tang-nano-9k-shield/GREEN -> RED
- R31 pad 1: /tang-nano-9k-shield/VGA_G0 -> /tang-nano-9k-shield/VGA_R0
- R31 pad 2: /tang-nano-9k-shield/GREEN -> RED
- U11 pad 32: unconnected-(U11-GPIO21-Pad32) -> /tang-nano-9k-shield/USB_PWR_EN
- U11 pad 36: unconnected-(U11-GPIO24-Pad36) -> /tang-nano-9k-shield/VBUS_DET
- U11 pad 37: unconnected-(U11-GPIO25-Pad37) -> /tang-nano-9k-shield/USB_FLT
- U12 pad 12: /tang-nano-9k-shield/PMOD10 -> /tang-nano-9k-shield/PMOD7
- U12 pad 13: /tang-nano-9k-shield/PMOD9 -> /tang-nano-9k-shield/PMOD8
- U12 pad 14: /tang-nano-9k-shield/PMOD8 -> /tang-nano-9k-shield/PMOD9
- U12 pad 15: /tang-nano-9k-shield/PMOD7 -> /tang-nano-9k-shield/PMOD10
- U12 pad 16: /tang-nano-9k-shield/PMOD4 -> /tang-nano-9k-shield/PMOD1
- U12 pad 17: /tang-nano-9k-shield/PMOD3 -> /tang-nano-9k-shield/PMOD2
- U12 pad 18: /tang-nano-9k-shield/PMOD2 -> /tang-nano-9k-shield/PMOD3
- U12 pad 20: /tang-nano-9k-shield/PMOD1 -> /tang-nano-9k-shield/PMOD4
- U2 pad 31: /tang-nano-9k-shield/PS/2_CLK2 -> /tang-nano-9k-shield/PS/2_DAT2
- U2 pad 32: /tang-nano-9k-shield/PS/2_DAT2 -> /tang-nano-9k-shield/PS/2_CLK2
- U2 pad 41: /tang-nano-9k-shield/VGA_R3 -> /tang-nano-9k-shield/VGA_G3
- U2 pad 42: /tang-nano-9k-shield/VGA_R2 -> /tang-nano-9k-shield/VGA_G2
- U2 pad 48: /tang-nano-9k-shield/PS/2_CLK1 -> /tang-nano-9k-shield/PS/2_DAT1
- U2 pad 49: /tang-nano-9k-shield/PS/2_DAT1 -> /tang-nano-9k-shield/PS/2_CLK1
- U2 pad 51: /tang-nano-9k-shield/VGA_R1 -> /tang-nano-9k-shield/VGA_G1
- U2 pad 53: /tang-nano-9k-shield/VGA_R0 -> /tang-nano-9k-shield/VGA_G0
- U2 pad 54: /tang-nano-9k-shield/VGA_G3 -> /tang-nano-9k-shield/VGA_R3
- U2 pad 55: /tang-nano-9k-shield/VGA_G2 -> /tang-nano-9k-shield/VGA_R2
- U2 pad 56: /tang-nano-9k-shield/VGA_G0 -> /tang-nano-9k-shield/VGA_R1
- U2 pad 57: /tang-nano-9k-shield/VGA_G1 -> /tang-nano-9k-shield/VGA_R0
- U9 pad 1: /tang-nano-9k-shield/RAW_D1+ -> /tang-nano-9k-shield/D1+
- U9 pad 3: /tang-nano-9k-shield/RAW_D1- -> /tang-nano-9k-shield/D1-
- U9 pad 4: /tang-nano-9k-shield/D1- -> /tang-nano-9k-shield/RAW_D1-
- U9 pad 5: 5V -> 5V_USB
- U9 pad 6: /tang-nano-9k-shield/D1+ -> /tang-nano-9k-shield/RAW_D1+

Commit message: Add files via upload
Parts:
- moved U8 153.6 mm to (60.2, 112.1), turned to 90 degrees
- moved R63 137.7 mm to (50.4, 97.9), turned to 180 degrees
- moved R64 136.2 mm to (53.7, 103.2), turned to 180 degrees
- moved R42 135.5 mm to (48.5, 112.4)
- moved C47 135.5 mm to (52.8, 99.8), turned to 180 degrees
- moved J6 134.7 mm to (44.9, 106.1), turned to -90 degrees
- moved R62 133.7 mm to (53.5, 97.9), turned to 180 degrees
- moved U13 130.8 mm to (57.3, 101.9), turned to 0 degrees
- moved R41 127.1 mm to (48.4, 99.9), turned to 0 degrees
- moved R61 126.6 mm to (61.0, 102.8), turned to 0 degrees
- moved C27 126.1 mm to (52.8, 108.7), turned to 0 degrees
- moved C46 125.3 mm to (61.0, 100.9), turned to 0 degrees
- moved U9 125.3 mm to (52.2, 106.1), turned to 180 degrees
- moved R60 125.1 mm to (55.6, 114.7)
- moved C45 124.5 mm to (61.1, 99.4), turned to 0 degrees
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
Commit message: Add files via upload
Parts:
- moved R19 122.4 mm to (98.9, 114.4), turned to -90 degrees
- moved R22 118.0 mm to (98.9, 111.2), turned to 90 degrees
- moved U3 113.1 mm to (132.9, 91.1), turned to 90 degrees
- moved U7 107.2 mm to (143.4, 102.9)
- moved D2 101.8 mm to (82.2, 107.2), turned to -90 degrees
- moved C5 93.5 mm to (149.2, 145.6), turned to 90 degrees
- moved L1 87.1 mm to (145.8, 90.0), turned to 180 degrees
- moved C1 73.8 mm to (131.0, 93.9), turned to 180 degrees
- moved C7 68.7 mm to (131.0, 88.2), turned to 180 degrees
- moved C21 66.6 mm to (131.1, 84.3), turned to 180 degrees
- moved C6 59.4 mm to (130.2, 86.3), turned to 180 degrees
- moved R24 58.2 mm to (150.8, 78.3), turned to 90 degrees
- moved D5 57.4 mm to (146.6, 143.6), turned to -90 degrees
- moved R25 57.1 mm to (151.5, 75.9)
- moved C23 56.7 mm to (146.2, 101.1), turned to 90 degrees
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Connections:
- net Net-(U11-USB_DM) renamed /tang-nano-9k-shield/USB_D-
- net Net-(U11-USB_DP) renamed /tang-nano-9k-shield/USB_D+
Routing:
- added copper zone on B.Cu, net GND
- added copper zone on F.Cu, net GND
- added copper zone on In1.Cu, net GND
- added copper zone on In2.Cu, net GND
Other:
- board outline added: 99.5 x 98.9 mm
- copper layers 2 -> 4

Commit message: Add files via upload
Parts:
- moved J2 6.17 mm to (84.0, 155.6)
- moved U9 0.89 mm to (81.0, 122.9)
- moved C27 0.86 mm to (81.6, 125.4)
- moved C37 0.29 mm to (96.7, 118.4)
- moved C28 0.24 mm to (90.3, 123.8)
- moved C48 0.24 mm to (90.3, 124.7)
- moved R49 0.23 mm to (108.3, 95.8)
- moved R6 0.23 mm to (147.7, 160.6)
- moved R48 0.23 mm to (111.3, 95.8)
- moved R5 0.23 mm to (147.7, 162.1)
- moved R47 0.22 mm to (114.4, 95.8)
- moved SW2 0.22 mm to (100.9, 89.0)
- moved R51 0.21 mm to (102.2, 95.8)
- moved R50 0.21 mm to (105.2, 95.8)
- moved R52 0.18 mm to (99.2, 95.8)
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Routing:
- net 5V_USB: track 0.00 -> 33.4 mm, vias 0 -> 5
- net /tang-nano-9k-shield/VBUS_DET: track 0.00 -> 24.4 mm, vias 0 -> 2
- net /tang-nano-9k-shield/USB_PWR_EN: track 0.00 -> 17.0 mm, vias 0 -> 2
- net 3V3: track 0.00 -> 16.7 mm
- net /tang-nano-9k-shield/USB_FLT: track 0.00 -> 16.0 mm, vias 0 -> 2
- net /tang-nano-9k-shield/SDA: track 0.00 -> 14.0 mm, vias 0 -> 1
- net /tang-nano-9k-shield/SCL: track 0.00 -> 10.8 mm
- net /tang-nano-9k-shield/XIN: track 0.00 -> 8.54 mm
- net /tang-nano-9k-shield/RAW_D1+: track 0.00 -> 6.43 mm
- net GND: track 0.00 -> 6.38 mm, vias 0 -> 52
- net /tang-nano-9k-shield/RAW_D1-: track 0.00 -> 6.34 mm
- net 5V_BUCK: track 0.00 -> 6.12 mm, vias 0 -> 2
- net /tang-nano-9k-shield/USB_D-: track 0.00 -> 5.71 mm
- net /tang-nano-9k-shield/USB_D+: track 0.00 -> 5.67 mm
- net /tang-nano-9k-shield/DVDD: track 0.00 -> 5.05 mm
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